Commit message: ref 103

File: urdf/Rover_Jonathan_Fisher.urdf (robot description, URDF)
Before this commit: robot Rover_Jonathan_Fisher, 17 links, 16 joints
Links:
- added link robot, mass 500.0; visual mesh filename=file://$(find robot_description)/meshes/dae/Cube.dae scale=1.0 1.715 0.78246
- link base_link: mass 500.0 -> None; geometry 
Joints:
- added joint base_link_joint: type fixed, parent base_link, child robot, origin xyz=0 0 0 rpy=0 0 1.57
- joint Barra_principal: parent base_link -> robot
- joint P_abajo: parent base_link -> robot
- joint P_atras: parent base_link -> robot
- joint P_derecha: parent base_link -> robot
- joint Untitled: parent base_link -> robot
- joint Untitled.001: parent base_link -> robot
- joint rueda1: parent base_link -> robot
- joint rueda2: parent base_link -> robot
- joint rueda3: parent base_link -> robot
- joint rueda4: parent base_link -> robot
