Commit message: Subiendo workspace

File: robot_description/urdf/Rover_Jonathan_Fisher.urdf (robot description, URDF)
Before this commit: robot Rover_Jonathan_Fisher, 18 links, 17 joints
Joints:
- removed joint Barra_pinza_fixed
- removed joint Barra_principal
- removed joint P_abajo
- removed joint P_atras
- removed joint P_derecha
- removed joint Pinza_L
- removed joint Pinza_R
- removed joint Untitled
- removed joint Untitled.001
- removed joint barra_fixed
- removed joint barra_sube_baja
- removed joint base_link_joint
- removed joint esfera
- removed joint rueda1
- removed joint rueda2
- removed joint rueda3
- removed joint rueda4
- added joint Barra_pinza_fixed_: type fixed, parent barra_sube_baja, child Barra_pinza_fixed, origin xyz=0 -0.01222 -0.7498 rpy=0 0 0
- added joint Barra_principal_: type prismatic, parent robot, child Barra_principal, origin xyz=0 -1.3 1.50313 rpy=0 0 0, axis 0 0 1.0, limit lower=-0.82 upper=0.5 effort=0 velocity=0
- added joint P_abajo_: type fixed, parent robot, child P_abajo, origin xyz=-0.13097 0.46899 -0.78586 rpy=0 0 0
- added joint P_atras_: type fixed, parent robot, child P_atras, origin xyz=0.00012 1.51088 0.10075 rpy=1.5708 0 0
- added joint P_derecha_: type fixed, parent robot, child P_derecha, origin xyz=-0.7846 0.50205 0.06662 rpy=1.5708 0 1.5708
- added joint Pinza_L_: type prismatic, parent Barra_pinza_fixed, child Pinza_L, origin xyz=-0.39871 0.01611 -0.26543 rpy=3.14159 1.5708 0, axis 0 0 1.0, limit lower=-0.2 upper=0 effort=0 velocity=0
- added joint Pinza_R_: type prismatic, parent Barra_pinza_fixed, child Pinza_R, origin xyz=0.44 0 -0.26 rpy=0 1.5708 0, axis 0 0 1.0, limit lower=-0.2 upper=0 effort=0 velocity=0
- added joint Untitled.001_: type fixed, parent robot, child Untitled.001, origin xyz=0.04728 -0.52958 0.01956 rpy=1.5708 0 0
- added joint Untitled_: type fixed, parent robot, child Untitled, origin xyz=0.81387 0.60732 -0.01647 rpy=0 1.5708 0
- added joint barra_fixed_: type fixed, parent esfera, child barra_fixed, origin xyz=0.03695 -0.02274 0.17047 rpy=1.5708 0 1.53837
- added joint barra_sube_baja_: type prismatic, parent barra_fixed, child barra_sube_baja, origin xyz=-1.83756 -0.82282 0.05342 rpy=-1.5708 -1.54235 0, axis 0 0 1.0, limit lower=-1.17 upper=0.9 effort=0 velocity=0
- added joint base_link_joint_: type fixed, parent base_link, child robot, origin xyz=0 0 0 rpy=0 0 1.57
- added joint esfera_: type continuous, parent Barra_principal, child esfera, origin xyz=-0.01713 0.0009 0.84188 rpy=0 0 0, axis 0 0 1.0, limit effort=0 velocity=0
- added joint rueda1_: type continuous, parent robot, child rueda1, origin xyz=1.5 1.47 -1.17 rpy=0 1.5708 0, axis 0 0 1.0, limit effort=0 velocity=0
- added joint rueda2_: type continuous, parent robot, child rueda2, origin xyz=1.5 -1.47 -1.17 rpy=0 1.5708 0, axis 0 0 1.0, limit effort=0 velocity=0
- added joint rueda3_: type continuous, parent robot, child rueda3, origin xyz=-1.5 1.47 -1.17 rpy=0 1.5708 0, axis 0 0 1.0, limit effort=0 velocity=0
- added joint rueda4_: type continuous, parent robot, child rueda4, origin xyz=-1.5 -1.47 -1.17 rpy=0 1.5708 0, axis 0 0 1.0, limit effort=0 velocity=0
