Commit message: roverB no va en gazebo

File: robot_description/urdf/roverB.urdf (robot description, URDF)
Before this commit: robot Rover_Jonathan_Fisher, 18 links, 17 joints
Links:
- removed link Barra_pinza_fixed
- removed link Barra_principal
- removed link Pinza_L
- removed link Pinza_R
- removed link barra_fixed
- removed link barra_sube_baja
- removed link esfera
- added link base_footprint
Joints:
- removed joint Barra_pinza_fixed_
- removed joint Barra_principal_
- removed joint Pinza_L_
- removed joint Pinza_R_
- removed joint barra_fixed_
- removed joint barra_sube_baja_
- removed joint esfera_
- added joint base_footprint_joint_: type fixed, parent base_footprint, child base_link, origin xyz=0 0 0 rpy=0 0 0

Commit message: va?

File: robot_description/urdf/roverB.urdf (robot description, URDF)
Before this commit: robot roverB, 12 links, 11 joints
Joints:
- joint base_footprint_joint_: origin xyz=0 0 0 rpy=0 0 0 -> xyz=0 0 1.5 rpy=0 0 0

Commit message: Añadido controlador

File: robot_description/urdf/roverB.urdf (robot description, URDF)
Before this commit: robot roverB, 12 links, 11 joints
Links:
- removed link rueda1
- removed link rueda2
- removed link rueda3
- removed link rueda4
- added link back_left_wheel_joint_, mass 10.0; collision mesh filename=file://$(find robot_description)/meshes/dae/Torus.001.dae scale=1.0 1.0 1.0; visual mesh filename=file://$(find robot_description)/meshes/dae/Torus.007.dae scale=0.4 0.4 1.0
- added link back_right_wheel_joint_, mass 10.0; collision mesh filename=file://$(find robot_description)/meshes/dae/Torus.004.dae scale=1.0 1.0 1.0; visual mesh filename=file://$(find robot_description)/meshes/dae/Torus.003.dae scale=0.4 0.4 1.0
- added link front_left_wheel_joint_, mass 10.0; collision mesh filename=file://$(find robot_description)/meshes/dae/Torus.000.dae scale=1.0 1.0 1.0; visual mesh filename=file://$(find robot_description)/meshes/dae/Torus.008.dae scale=0.4 0.4 1.0
- added link front_right_wheel_joint_, mass 10.0; collision mesh filename=/$(find robot_description)/meshes/dae/Torus.002.dae scale=1.0 1.0 1.0; visual mesh filename=file://$(find robot_description)/meshes/dae/Torus.006.dae scale=0.4 0.4 1.0
Joints:
- removed joint rueda1_
- removed joint rueda2_
- removed joint rueda3_
- removed joint rueda4_
- added joint back_left_wheel_joint: type continuous, parent robot, child back_left_wheel_joint_, origin xyz=1.5 1.47 -1.17 rpy=0 1.5708 0, axis 0 0 1.0, limit effort=0 velocity=0
- added joint back_right_wheel_joint: type continuous, parent robot, child back_right_wheel_joint_, origin xyz=-1.5 1.47 -1.17 rpy=0 1.5708 3.1416, axis 0 0 1.0, limit effort=0 velocity=0
- added joint front_left_wheel_joint: type continuous, parent robot, child front_left_wheel_joint_, origin xyz=1.5 -1.47 -1.17 rpy=0 1.5708 0, axis 0 0 1.0, limit effort=0 velocity=0
- added joint front_right_wheel_joint: type continuous, parent robot, child front_right_wheel_joint_, origin xyz=-1.5 -1.47 -1.17 rpy=0 1.5708 3.1416, axis 0 0 1.0, limit effort=0 velocity=0
